File: PCB+schematic/logan.kicad_pcb (KiCad board)
At the start: 2 copper layers, 63 x 50.5 mm, 7 parts, among them J1 Arduino DC Jack (6-12v)

Commit message: kicad
Parts:
- added J2: SD Card, Connector_PinHeader_2.54mm:PinHeader_1x06_P2.54mm_Vertical, F.Cu at (165.0, 104.5)
- added J3: BME280, Connector_PinHeader_2.54mm:PinHeader_1x04_P2.54mm_Vertical, F.Cu at (167.0, 78.4)
- added J4: LoRa, Connector_PinHeader_2.54mm:PinHeader_1x09_P2.54mm_Vertical, F.Cu at (111.2, 98.5)
- added J5: LoRa G pins, Connector_PinHeader_2.54mm:PinHeader_1x05_P2.54mm_Vertical, F.Cu at (111.2, 73.5)
- moved H2 16.2 mm to (184.5, 76.0)
- moved H4 16.0 mm to (184.5, 121.0)
- moved H1 11.4 mm to (102.5, 75.5)
- moved H3 11.0 mm to (102.0, 121.0)
Connections:
- A1 pad 14: /D11 -> /MOSI
- A1 pad 15: /D12 -> /MISO
- A1 pad 16: /D13 -> /SCK
- A1 pad 23: /A4 -> /BME_SDA
- A1 pad 24: /A5 -> /BME_SCL
- A1 pad 5: /D2 -> /LORA_RST
- A1 pad 6: /D3 -> /G0
- A1 pad 7: /D4 -> /LORA_CS
- A1 pad 8: /D5 -> /SD_CS
Other:
- board size 63 x 50.5 mm -> 91.5 x 54 mm

Commit message: update PCB
Routing:
- net /SCK: track 0.00 -> 71.4 mm
- net /MOSI: track 0.00 -> 67.8 mm
- net +5V: track 0.00 -> 66.6 mm
- net /MISO: track 0.00 -> 64.4 mm, vias 0 -> 2
- net /NANO_VIN: track 0.00 -> 42.0 mm
- net /SD_CS: track 0.00 -> 37.0 mm
- net +3.3V: track 0.00 -> 33.8 mm
- net /G0: track 0.00 -> 22.4 mm
- net /BME_SDA: track 0.00 -> 21.2 mm
- net /BME_SCL: track 0.00 -> 21.0 mm
- net /~{RESET}: track 0.00 -> 15.2 mm
- net /LORA_CS: track 0.00 -> 12.2 mm
- net /LORA_RST: track 0.00 -> 10.8 mm, vias 0 -> 1
- net Earth: track 0.00 -> 7.37 mm, vias 0 -> 1
- added copper zone on F.Cu, net Earth
Other:
- board text added: "By Logan Caramanna"
