File: PCB+schematic/logan.kicad_sch (KiCad schematic)
At the start: 6 parts, among them J1 Arduino DC Jack (6-12v)

Commit message: pcb stuff
Parts:
- added J2: SD Card, Connector_PinHeader_2.54mm:PinHeader_1x06_P2.54mm_Vertical, symbol Connector:Conn_01x06_Socket
- added J3: BME280, Connector_PinHeader_2.54mm:PinHeader_1x04_P2.54mm_Vertical, symbol Connector:Conn_01x04_Socket
- added J4: LoRa, Connector_PinHeader_2.54mm:PinHeader_1x09_P2.54mm_Vertical, symbol Connector:Conn_01x09_Socket
Connections:
- net +3.3V: now also J2.6 (Pin_6)
- net +5V: now also J3.1 (Pin_1), J4.1 (Pin_1)
- net Earth: now also J2.1 (Pin_1), J3.2 (Pin_2), J4.2 (Pin_2)
- net A4 renamed BME_SDA
- net BME_SDA: now also J3.4 (Pin_4)
- net A5 renamed BME_SCL
- net BME_SCL: now also J3.3 (Pin_3)
- net D11 renamed MOSI
- net MOSI: now also J2.4 (Pin_4)
- net D12 renamed MISO
- net MISO: now also J2.2 (Pin_2), J4.6 (Pin_6)
- net D13 renamed SCK
- net SCK: now also J2.3 (Pin_3), J4.5 (Pin_5)
- net D2 renamed LORA_RST
- net LORA_RST: now also J4.9 (Pin_9)
- net D3 renamed G0
- net G0: now also J4.4 (Pin_4)
- net D4 renamed LORA_CS
- net LORA_CS: now also J4.8 (Pin_8)
- net D5 renamed SD_CS
- net SD_CS: now also J2.5 (Pin_5)
- new net SD_MOSI: J4.7 (Pin_7)
Other:
- note removed: "Please place any sensor symbols you want in this block. Please feel free to extend the box's bounds to fit everything! (Delete this after!)"
- note removed: "SD Card or external memory chip. (Delete this after!)"
- title: My StratoScience Project Name (double-click here to edit) -> LoRa thingy

Commit message: kicad
Parts:
- added J5: LoRa G pins, Connector_PinHeader_2.54mm:PinHeader_1x05_P2.54mm_Vertical, symbol Connector:Conn_01x05_Socket
Connections:
- net SD_MOSI is gone; now on net MOSI: J4.7 (Pin_7)
- no-connect marks 0 -> 6
Changed lines of the file:
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@@
 		(color 0 0 0 0)
 	)
+	(no_connect
+		(at 137.16 121.92)
+	)
+	(no_connect
+		(at 137.16 124.46)
+	)
+	(no_connect
+		(at 137.16 119.38)
+	)
+	(no_connect
+		(at 137.16 127)
+	)
+	(no_connect
+		(at 161.29 96.52)
+	)
+	(no_connect
+		(at 137.16 129.54)
+	)
 	(wire
 		(pts
@@
 	(wire
 		(pts
+			(xy 161.29 96.52) (xy 163.83 96.52)
+		)
+		(stroke
+			(width 0)
+			(type default)
+		)
+	)
+	(wire
+		(pts
 			(xy 151.13 92.71) (xy 151.13 100.33)
 		)
@@
 	(wire
 		(pts
+			(xy 137.16 127) (xy 139.7 127)
+		)
+		(stroke
+			(width 0)
+			(type default)
+		)
+	)
+	(wire
+		(pts
+			(xy 137.16 124.46) (xy 139.7 124.46)
+		)
+		(stroke
+			(width 0)
+			(type default)
+		)
+	)
+	(wire
+		(pts
 			(xy 187.96 93.98) (xy 195.58 93.98)
 		)
@@
 	(wire
 		(pts
+			(xy 137.16 129.54) (xy 139.7 129.54)
+		)
+		(stroke
+			(width 0)
+			(type default)
+		)
+	)
+	(wire
+		(pts
 			(xy 163.83 95.25) (xy 152.4 95.25)
 		)
@@
 	(wire
 		(pts
+			(xy 163.83 96.52) (xy 163.83 97.79)
+		)
+		(stroke
+			(width 0)
+			(type default)
+		)
+	)
+	(wire
+		(pts
 			(xy 130.81 100.33) (xy 133.35 100.33)
 		)
@@
 	(wire
 		(pts
+			(xy 137.16 121.92) (xy 139.7 121.92)
+		)
+		(stroke
+			(width 0)
+			(type default)
+		)
+	)
+	(wire
+		(pts
 			(xy 133.35 78.74) (xy 144.78 78.74)
 		)
@@
 		(pts
 			(xy 132.08 113.03) (xy 140.97 113.03)
+		)
+		(stroke
+			(width 0)
+			(type default)
+		)
+	)
+	(wire
+		(pts
+			(xy 137.16 119.38) (xy 139.7 119.38)
 		)
 		(stroke
@@
 		)
 	)
-	(label "SD_MOSI"
+	(label "MOSI"
 		(at 162.56 107.95 180)
 		(fields_autoplaced yes)
@@
 					(unit 1)
 				)
+			)
+		)
+	)
+	(symbol
+		(lib_id "Connector:Conn_01x05_Socket")
+		(at 144.78 124.46 0)
+		(unit 1)
+		(exclude_from_sim no)
+		(in_bom yes)
+		(on_board yes)
+		(dnp no)
+		(fields_autoplaced yes)
+		(property "Reference" "J5"
+			(at 146.05 123.1899 0)
+			(effects
+				(font
+					(size 1.27 1.27)
+				)
+				(justify left)
+			)
+		)
+		(property "Value" "LoRa G pins"
+			(at 146.05 125.7299 0)
+			(effects
+				(font
+					(size 1.27 1.27)
+				)
+				(justify left)
+			)
+		)
+		(property "Footprint" "Connector_PinHeader_2.54mm:PinHeader_1x05_P2.54mm_Vertical"
+			(at 144.78 124.46 0)
+			(effects
+				(font
+					(size 1.27 1.27)
+				)
+				(hide yes)
+			)
+		)
+		(property "Datasheet" "~"
+			(at 144.78 124.46 0)
+			(effects
+				(font
+					(size 1.27 1.27)
+				)
+				(hide yes)
+			)
+		)
+		(property "Description" "Generic connector, single row, 01x05, script generated"
+			(at 144.78 124.46 0)
+			(effects
+				(font
+					(size 1.27 1.27)
+				)
+				(hide yes)
+			)
+		)
+		(pin "1"
+		)
+		(pin "2"
+		)
+		(pin "5"
+		)
+		(pin "4"
+		)
+		(pin "3"
+		)
+		(instances
+			(project ""
+				(path "/b7aacd66-2173-43d2-8b45-08f19cb7b7f8"
+					(reference "J5")
+					(unit 1)
+				)

Commit message: update PCB
Changed lines of the file:
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@@
 (kicad_sch
-	(version 20231120)
+	(version 20250114)
 	(generator "eeschema")
-	(generator_version "8.0")
+	(generator_version "9.0")
 	(paper "A4")
 	(title_block
@@
 		(comment 1 "by Logan Caramanna")
 	)
+	(rectangle
+		(start 175.26 58.42)
+		(end 220.98 130.81)
+		(stroke
+			(width 0)
+			(type default)
+		)
+		(fill
+			(type none)
+		)
+	)
+	(rectangle
+		(start 220.98 99.06)
+		(end 247.65 130.81)
+		(stroke
+			(width 0)
+			(type default)
+		)
+		(fill
+			(type none)
+		)
+	)
+	(rectangle
+		(start 128.27 58.42)
+		(end 175.26 90.17)
+		(stroke
+			(width 0)
+			(type default)
+		)
+		(fill
+			(type none)
+		)
+	)
+	(rectangle
+		(start 128.27 90.17)
+		(end 175.26 130.81)
+		(stroke
+			(width 0)
+			(type default)
+		)
+		(fill
+			(type none)
+		)
+	)
+	(rectangle
+		(start 69.85 58.42)
+		(end 128.27 130.81)
+		(stroke
+			(width 0)
+			(type default)
+		)
+		(fill
+			(type none)
+		)
+	)
+	(text "Data Logging"
+		(exclude_from_sim no)
+		(at 182.626 60.706 0)
+		(effects
+			(font
+				(size 1.27 1.27)
+			)
+		)
+	)
+	(text "Custom Sensors"
+		(exclude_from_sim no)
+		(at 137.16 93.218 0)
+		(effects
+			(font
+				(size 1.27 1.27)
+			)
+		)
+	)
+	(text "Power Input"
+		(exclude_from_sim no)
+		(at 134.874 60.706 0)
+		(effects
+			(font
+				(size 1.27 1.27)
+			)
+		)
+	)
+	(text "Arduino Nano"
+		(exclude_from_sim no)
+		(at 77.216 60.96 0)
+		(effects
+			(font
+				(size 1.27 1.27)
+			)
+		)
+	)
+	(text "Placeholder text is optional. Feel free to adapt this sheet to better suit your project!"
+		(exclude_from_sim no)
+		(at 146.05 134.874 0)
+		(effects
+			(font
+				(size 1.27 1.27)
+			)
+		)
+	)
+	(text "Mounting Holes"
+		(exclude_from_sim no)
+		(at 229.362 101.854 0)
+		(effects
+			(font
+				(size 1.27 1.27)
+			)
+		)
+	)
 	(junction
 		(at 96.52 120.65)
@@
 		)
 	)
-	(rectangle
-		(start 175.26 58.42)
-		(end 220.98 130.81)
-		(stroke
-			(width 0)
-			(type default)
-		)
-		(fill
-			(type none)
-		)
-	)
-	(rectangle
-		(start 220.98 99.06)
-		(end 247.65 130.81)
-		(stroke
-			(width 0)
-			(type default)
-		)
-		(fill
-			(type none)
-		)
-	)
-	(rectangle
-		(start 128.27 58.42)
-		(end 175.26 90.17)
-		(stroke
-			(width 0)
-			(type default)
-		)
-		(fill
-			(type none)
-		)
-	)
-	(rectangle
-		(start 128.27 90.17)
-		(end 175.26 130.81)
-		(stroke
-			(width 0)
-			(type default)
-		)
-		(fill
-			(type none)
-		)
-	)
-	(rectangle
-		(start 69.85 58.42)
-		(end 128.27 130.81)
-		(stroke
-			(width 0)
-			(type default)
-		)
-		(fill
-			(type none)
-		)
-	)
-	(text "Data Logging"
-		(exclude_from_sim no)
-		(at 182.626 60.706 0)
-		(effects
-			(font
-				(size 1.27 1.27)
-			)
-		)
-	)
-	(text "Custom Sensors"
-		(exclude_from_sim no)
-		(at 137.16 93.218 0)
-		(effects
-			(font
-				(size 1.27 1.27)
-			)
-		)
-	)
-	(text "Power Input"
-		(exclude_from_sim no)
-		(at 134.874 60.706 0)
-		(effects
-			(font
-				(size 1.27 1.27)
-			)
-		)
-	)
-	(text "Arduino Nano"
-		(exclude_from_sim no)
-		(at 77.216 60.96 0)
-		(effects
-			(font
-				(size 1.27 1.27)
-			)
-		)
-	)
-	(text "Placeholder text is optional. Feel free to adapt this sheet to better suit your project!"
-		(exclude_from_sim no)
-		(at 146.05 134.874 0)
-		(effects
-			(font
-				(size 1.27 1.27)
-			)
-		)
-	)
-	(text "Mounting Holes"
-		(exclude_from_sim no)
-		(at 229.362 101.854 0)
-		(effects
-			(font
-				(size 1.27 1.27)
-			)
-		)
-	)
 	(label "BME_SCL"
 		(at 132.08 113.03 0)
-		(fields_autoplaced yes)
 		(effects
 			(font
@@
 	(label "D0/RX"
 		(at 83.82 80.01 180)
-		(fields_autoplaced yes)
 		(effects
 			(font
@@
 	(label "D9"
 		(at 83.82 102.87 180)
-		(fields_autoplaced yes)
 		(effects
 			(font
@@
 	(label "A1"
 		(at 109.22 97.79 0)
-		(fields_autoplaced yes)
 		(effects
 			(font
@@
 	(label "MOSI"
 		(at 187.96 96.52 0)
-		(fields_autoplaced yes)
 		(effects
 			(font
@@
 	(label "D1/TX"
 		(at 83.82 82.55 180)
-		(fields_autoplaced yes)
 		(effects
 			(font
@@
 	(label "LORA_CS"
 		(at 83.82 90.17 180)
-		(fields_autoplaced yes)
 		(effects
 			(font
@@
 	(label "SCK"
 		(at 162.56 102.87 180)
-		(fields_autoplaced yes)
 		(effects
 			(font
@@
 	(label "LORA_RST"
 		(at 162.56 113.03 180)
-		(fields_autoplaced yes)
 		(effects
 			(font
@@
 	(label "~{RESET}"
 		(at 109.22 80.01 0)
-		(fields_autoplaced yes)
 		(effects
 			(font
@@
 	(label "MOSI"
 		(at 162.56 107.95 180)
-		(fields_autoplaced yes)
 		(effects
 			(font
@@
 	(label "SD_CS"
 		(at 187.96 99.06 0)
-		(fields_autoplaced yes)
 		(effects
 			(font
@@
 	(label "A6"
 		(at 109.22 110.49 0)
-		(fields_autoplaced yes)
 		(effects
 			(font
@@
 	(label "D10"
 		(at 83.82 105.41 180)
-		(fields_autoplaced yes)
 		(effects
 			(font
@@
 	(label "LORA_RST"
 		(at 83.82 85.09 180)
-		(fields_autoplaced yes)
 		(effects
 			(font
@@
 	(label "SCK"
 		(at 187.96 93.98 0)
-		(fields_autoplaced yes)
 		(effects
 			(font
@@
 	(label "A2"
 		(at 109.22 100.33 0)
-		(fields_autoplaced yes)
 		(effects
 			(font
@@
 	(label "NANO_VIN"
 		(at 133.35 78.74 0)
-		(fields_autoplaced yes)
 		(effects
 			(font
@@
 	(label "A7"
 		(at 109.22 113.03 0)
-		(fields_autoplaced yes)
 		(effects
 			(font
@@
 	(label "D7"
 		(at 83.82 97.79 180)
-		(fields_autoplaced yes)
 		(effects
 			(font
@@
 	(label "BME_SDA"
 		(at 132.08 115.57 0)
-		(fields_autoplaced yes)
 		(effects
 			(font
@@
 	(label "MISO"
 		(at 162.56 105.41 180)
-		(fields_autoplaced yes)
 		(effects
 			(font
@@
 	(label "AREF"
 		(at 109.22 90.17 0)
-		(fields_autoplaced yes)
 		(effects
 			(font
@@
 	(label "A3"
 		(at 109.22 102.87 0)
-		(fields_autoplaced yes)
 		(effects
 			(font
@@
 	(label "MOSI"
 		(at 83.82 107.95 180)
-		(fields_autoplaced yes)
 		(effects
 			(font
@@
 	(label "G0"
 		(at 83.82 87.63 180)
-		(fields_autoplaced yes)
 		(effects
 			(font
@@
 	(label "D8"
 		(at 83.82 100.33 180)
-		(fields_autoplaced yes)
 		(effects
 			(font
@@
 	(label "NANO_VIN"
 		(at 93.98 68.58 180)
-		(fields_autoplaced yes)
 		(effects
 			(font
@@
 	(label "SD_CS"
 		(at 83.82 92.71 180)
-		(fields_autoplaced yes)
 		(effects
 			(font
@@
 	(label "A0"
 		(at 109.22 95.25 0)
-		(fields_autoplaced yes)
 		(effects
 			(font
@@
 	(label "MISO"
 		(at 83.82 110.49 180)
-		(fields_autoplaced yes)
 		(effects
 			(font
@@
 	(label "LORA_CS"
 		(at 162.56 110.49 180)
-		(fields_autoplaced yes)
 		(effects
 			(font
@@
 	(label "D6"
 		(at 83.82 95.25 180)
-		(fields_autoplaced yes)
 		(effects
 			(font
@@
 	(label "~{RESET}"
 		(at 109.22 82.55 0)
-		(fields_autoplaced yes)
 		(effects
 			(font
@@
 	(label "BME_SCL"
 		(at 109.22 107.95 0)
-		(fields_autoplaced yes)
 		(effects
 			(font
@@
 	(label "SCK"
 		(at 83.82 113.03 180)
-		(fields_autoplaced yes)
 		(effects
 			(font
@@
 	(label "G0"
 		(at 162.56 100.33 180)
-		(fields_autoplaced yes)
 		(effects
 			(font
@@
 	(label "BME_SDA"
 		(at 109.22 105.41 0)
-		(fields_autoplaced yes)
 		(effects
 			(font
@@
 	(label "MISO"
 		(at 187.96 91.44 0)
-		(fields_autoplaced yes)
 		(effects
 			(font
@@
 		)
 	)
+	(embedded_fonts no)
 )
